File: hardware/LUMISPARK-300X.kicad_sch (KiCad schematic)
At the start: 22 parts, among them J1 2-Pad AC In (L & N), J2 2-Pad Output (+ & -), Q1 BT136-600, SW1 SW_SPST, SW2 SW_SPST

Commit message: Uploaded all latest files
Parts:
- added RV3: 500kΩ Potentiometer, Connector_Wire:SolderWire-0.5sqmm_1x03_P4.6mm_D0.9mm_OD2.1mm, symbol Device:R_Potentiometer
- added R_CAL1: 4.7kΩ 1W, Resistor_THT:R_Axial_DIN0411_L9.9mm_D3.6mm_P15.24mm_Horizontal, symbol Device:R
Connections:
- net AC_PHASE_OUT: now also RV3.3
- net at R_LDR1.1, SW1.2 (B): now also R_CAL1.1
- new net: RV3.1, RV3.2, R_CAL1.2
